File: usbtinyisp.brd (EAGLE design)
At the start: 24.6 x 12.2 mm, 9 parts

Commit message: via/pours fix
Routing:
- net GND: track 5.72 -> 4.21 mm, vias 6 -> 9
Changed lines of the file:
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@@
 <setting verticaltext="up"/>
 </settings>
-<grid distance="1" unitdist="mil" unit="mil" style="lines" multiple="1" display="yes" altdistance="0.025" altunitdist="inch" altunit="inch"/>
+<grid distance="10" unitdist="mil" unit="mil" style="lines" multiple="1" display="yes" altdistance="0.025" altunitdist="inch" altunit="inch"/>
 <layers>
 <layer number="1" name="Top" color="4" fill="1" visible="yes" active="yes"/>
@@
 <contactref element="U$1" pad="GND"/>
 <contactref element="JP2" pad="6"/>
-<via x="10.668" y="15.748" extent="1-16" drill="0.2032" diameter="0.4572"/>
-<via x="17.018" y="15.748" extent="1-16" drill="0.2032" diameter="0.4572"/>
+<via x="18.288" y="16.51" extent="1-16" drill="0.2032" diameter="0.4572"/>
 <wire x1="5.388" y1="14.676" x2="9.596" y2="14.676" width="0.4064" layer="1"/>
-<wire x1="9.596" y1="14.676" x2="10.668" y2="15.748" width="0.4064" layer="1"/>
 <via x="11.684" y="7.874" extent="1-16" drill="0.2032"/>
 <via x="13.208" y="5.842" extent="1-16" drill="0.2032"/>
 <via x="15.748" y="6.858" extent="1-16" drill="0.2032"/>
 <via x="22.606" y="16.002" extent="1-16" drill="1.2"/>
+<via x="18.288" y="5.842" extent="1-16" drill="0.2032" diameter="0.4572"/>
+<via x="24.384" y="11.176" extent="1-16" drill="0.2032" diameter="0.4572"/>
+<via x="13.208" y="16.51" extent="1-16" drill="0.2032" diameter="0.4572"/>
+<via x="9.652" y="16.51" extent="1-16" drill="0.2032" diameter="0.4572"/>
 </signal>
 <signal name="N$3">
